File: hardware/Pleasc.kicad_pcb (KiCad board)
At the start: 6 copper layers, 60 x 60 mm, 133 parts, among them J1 5023860570, J2 2601-1104, J3 2601-1104, J4 39-29-1048, J6 ESQ-110-14-G-D, Q1 AO3400A, Q10 AO3400A, Q11 AO3400A, Q12 AO3400A, Q13 AO3400A, Q14 AO3400A, Q2 AO3400A, Q3 AO3400A, Q4 AO3400A, Q5 AO3400A, Q6 AO3400A, Q7 AO3400A, Q8 AO3400A, Q9 AO3400A, U1 LTV-817, U10 STM32F072C8Tx, U11 TJA1051T-3, U12 MPM3650CGQW-P, U13 TLV75533PDRV, U2 LTV-817, U3 LTV-817, U4 LTV-817, U5 LTV-817, U6 LTV-817, U7 LTV-817, U8 LTV-817, U9 LTV-817

Commit message: ready 2 order
Parts:
- renumbered 3.3V1 to 3.3V, 5V1 to 5V, CAN+1 to CAN+, CAN-1 to CAN-, GND1 to GND, PGND1 to PGND, PYRO_ON1 to PYRO_ON, VBAT1 to VBAT
Routing:
- net 3.3V: track 155.7 -> 161.4 mm
- added copper zone on In1.Cu, net GND
- added copper zone on In4.Cu, net GND
Changed lines of the file:
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@@
 		(layer "F.Cu")
 		(at 84.5 83.5)
-		(property "Reference" "PYRO_ON1"
+		(property "Reference" "PYRO_ON"
 			(at 1.5 -1.5 0)
 			(layer "F.SilkS")
@@
 		(layer "F.Cu")
 		(at 87.54 67.02)
-		(property "Reference" "CAN-1"
+		(property "Reference" "CAN-"
 			(at -0.91 1.43 0)
 			(layer "F.SilkS")
@@
 		(layer "F.Cu")
 		(at 90.75 86.5)
-		(property "Reference" "VBAT1"
+		(property "Reference" "VBAT"
 			(at 0 -1.48 0)
 			(layer "F.SilkS")
@@
 		(layer "F.Cu")
 		(at 87.92 63.44 90)
-		(property "Reference" "CAN+1"
+		(property "Reference" "CAN+"
 			(at 3.12 0.04 270)
 			(layer "F.SilkS")
@@
 		(layer "F.Cu")
 		(at 84.25 86.5)
-		(property "Reference" "3.3V1"
+		(property "Reference" "3.3V"
 			(at 0 -1.5 0)
 			(layer "F.SilkS")
@@
 		(layer "F.Cu")
 		(at 87.476886 86.5 180)
-		(property "Reference" "5V1"
+		(property "Reference" "5V"
 			(at 0 1.5 180)
 			(layer "F.SilkS")
@@
 		(layer "F.Cu")
 		(at 80.943489 83.5)
-		(property "Reference" "PGND1"
+		(property "Reference" "PGND"
 			(at -0.06 -1.5 0)
 			(layer "F.SilkS")
@@
 		(layer "F.Cu")
 		(at 81 86.5)
-		(property "Reference" "GND1"
+		(property "Reference" "GND"
 			(at -0.01 -1.5 0)
 			(layer "F.SilkS")
@@
 	)
 	(segment
+		(start 63.25 60.5)
+		(end 65.75 60.5)
+		(width 0.2)
+		(layer "In2.Cu")
+		(net 1)
+	)
+	(segment
 		(start 70 45.575)
 		(end 70.425 45.575)
@@
 	)
 	(segment
-		(start 68.17 58.39)
+		(start 68.015 58.235)
 		(end 63.31 53.53)
 		(width 0.4)
@@
 	)
 	(segment
+		(start 65.75 60.5)
+		(end 68.015 58.235)
+		(width 0.2)
+		(layer "In2.Cu")
+		(net 1)
+	)
+	(segment
 		(start 84.105144 53.824856)
 		(end 82.03 55.9)
@@
 	)
 	(segment
+		(start 68.17 58.39)
+		(end 68.015 58.235)
+		(width 0.4)
+		(layer "In2.Cu")
+		(net 1)
+	)
+	(segment
 		(start 63.31 53.53)
 		(end 63.31 53.05)
@@
 		(net 2)
 		(net_name "GND")
-		(layers "F.Cu" "B.Cu" "In2.Cu" "In3.Cu")
+		(layers "F.Cu" "B.Cu" "In1.Cu" "In2.Cu" "In3.Cu" "In4.Cu")
 		(hatch edge 0.5)
 		(connect_pads
