File: hardware/Pleasc.kicad_pcb (KiCad board)
At the start: 6 copper layers, 60 x 60 mm, 133 parts, among them J1 5023860570, J2 2601-1104, J3 2601-1104, J4 39-29-1048, J6 ESQ-110-14-G-D, Q1 AO3400A, Q10 AO3400A, Q11 AO3400A, Q12 AO3400A, Q13 AO3400A, Q14 AO3400A, Q2 AO3400A, Q3 AO3400A, Q4 AO3400A, Q5 AO3400A, Q6 AO3400A, Q7 AO3400A, Q8 AO3400A, Q9 AO3400A, U1 LTV-817, U10 STM32F072C8Tx, U11 TJA1051T-3, U12 MPM3650CGQW-P, U13 TLV75533PDRV, U2 LTV-817, U3 LTV-817, U4 LTV-817, U5 LTV-817, U6 LTV-817, U7 LTV-817, U8 LTV-817, U9 LTV-817

Commit message: hardware done
Parts:
- added G***: LOGO, LOGO, F.Cu at (94.9, 81.1)
- C14, C17, C20, C23, C24, C25, C27, C28, C29: footprint Capacitor_SMD:C_0402_1005Metric -> Capacitor_SMD:C_0603_1608Metric
- moved C30 5.65 mm to (84.3, 46.3), turned to 0 degrees
- moved C22 3.01 mm to (82.9, 30.0)
- moved C25 0.85 mm to (81.8, 46.1)
- moved C23 0.74 mm to (82.9, 32.8)
- moved C29 0.71 mm to (81.9, 41.5)
- moved C16 0.67 mm to (82.0, 54.8)
- moved D10 0.65 mm to (85.4, 62.8)
- moved R9 0.60 mm to (82.2, 58.5), turned to -90 degrees
- moved R40 0.43 mm to (86.7, 59.5)
- moved R41 0.42 mm to (84.1, 59.5)
- moved C14 0.37 mm to (68.0, 55.0)
- moved C17 0.33 mm to (85.3, 48.9)
- moved C27 0.31 mm to (81.9, 44.5)
- moved C20 0.27 mm to (85.4, 59.5)
- moved C24 0.24 mm to (82.9, 31.2)
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- renumbered 3.3V to 3V3, PYRO_ON to PON
Routing:
- net 5VLOGIC: track 110.5 -> 90.1 mm, vias 7 -> 4
- net PGND: track 175.8 -> 179.0 mm
- net DROGUE_FIRE: track 16.7 -> 15.3 mm
- net SWDIO: track 26.5 -> 27.8 mm
- net CAN_o-: track 15.2 -> 16.3 mm
- net CAN_o+: track 16.8 -> 17.7 mm
- net CAN_+: track 12.0 -> 12.8 mm
- net CAN_-: track 11.9 -> 12.7 mm
- net 3.3V: track 161.4 -> 160.7 mm
- net Net-(R9-Pad2): track 1.80 -> 1.17 mm
- net Net-(C20-Pad1): track 1.95 -> 2.56 mm
- net GND: track 38.4 -> 38.7 mm, vias 97 -> 98
