File: hardware/power.kicad_sch (KiCad schematic)
At the start: 17 parts, among them U2 MPM3650CGQW-P, U5 TLV75533PDRV

Commit message: ready for review the twost
Parts:
- added C11, C12: 4.7uf, Capacitor_SMD:C_0402_1005Metric, symbol Device:C
- added C13: 10uf, Capacitor_SMD:C_0402_1005Metric, symbol Device:C
- added R7: 33.2kΩ, Resistor_SMD:R_0402_1005Metric, symbol Device:R
- added VR?: LT3045EDD_PBF, SON50P300X300X80-11N, symbol LT3045EDD_PBF:LT3045EDD_PBF
Connections:
- net GND: now also C11.1, C12.1, C13.2, R7.2, VR?.11 (EXP), VR?.5 (ILIM), VR?.8 (GND)
- net at C10.1, C21.1, C34.1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: now also C12.2, VR?.1 (IN_1), VR?.2 (IN_2), VR?.3 (EN/UV), VR?.6 (PGFB)
- new net: C11.2, R7.1, VR?.7 (SET)
- new net 3V3RF: C13.1, VR?.10 (OUT), VR?.9 (OUTS)
- no-connect marks 7 -> 8
Other:
- note removed: "what value should these caps be?"

Commit message: ready 2 order
Parts:
- removed C11, C12: 4.7uf, Capacitor_SMD:C_0402_1005Metric, symbol Device:C
- removed C13: 10uf, Capacitor_SMD:C_0402_1005Metric, symbol Device:C
- removed R7: 33.2kΩ, Resistor_SMD:R_0402_1005Metric, symbol Device:R
- removed VR?: LT3045EDD_PBF, SON50P300X300X80-11N, symbol LT3045EDD_PBF:LT3045EDD_PBF
- renumbered C10 to C21, C11 to C22, C29 to C23, C19 to C24, C48 to C25, C20 to C26, C47 to C27, C35 to C28, C34 to C29, C21 to C30, C50 to C31, C51 to C34, R3 to R42, R4 to R43, R7 to R44, U2 to U12, U5 to U13
Connections:
- no-connect marks 8 -> 7

Commit message: hardware done
Parts:
- C23, C24, C25, C27, C28, C29: footprint Capacitor_SMD:C_0402_1005Metric -> Capacitor_SMD:C_0603_1608Metric
Changed lines of the file:
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@@
 			)
 		)
-		(property "Footprint" "Capacitor_SMD:C_0402_1005Metric"
+		(property "Footprint" "Capacitor_SMD:C_0603_1608Metric"
 			(at 96.8248 105.41 0)
 			(effects
@@
 			)
 		)
-		(property "Footprint" "Capacitor_SMD:C_0402_1005Metric"
+		(property "Footprint" "Capacitor_SMD:C_0603_1608Metric"
 			(at 159.7152 90.17 0)
 			(effects
@@
 			)
 		)
-		(property "Footprint" "Capacitor_SMD:C_0402_1005Metric"
+		(property "Footprint" "Capacitor_SMD:C_0603_1608Metric"
 			(at 172.4152 90.17 0)
 			(effects
@@
 			)
 		)
-		(property "Footprint" "Capacitor_SMD:C_0402_1005Metric"
+		(property "Footprint" "Capacitor_SMD:C_0603_1608Metric"
 			(at 178.7652 90.17 0)
 			(effects
@@
 			)
 		)
-		(property "Footprint" "Capacitor_SMD:C_0402_1005Metric"
+		(property "Footprint" "Capacitor_SMD:C_0603_1608Metric"
 			(at 103.1748 105.41 0)
 			(effects
@@
 			)
 		)
-		(property "Datasheet" "~"
+		(property "Datasheet" ""
 			(at 104.14 109.22 0)
 			(effects
@@
 			)
 		)
-		(property "Footprint" "Capacitor_SMD:C_0402_1005Metric"
+		(property "Footprint" "Capacitor_SMD:C_0603_1608Metric"
 			(at 166.0652 90.17 0)
 			(effects
